File: eagle/can4vscp_usb_rev_B.brd (EAGLE design)
At the start: 72 x 42.6 mm, 29 parts, among them IC1 PIC18LF2550-I/SO, IC2 MCP2515, IC3 MCP2551SN, IC4 ISO1050, IC5 DCDC_MER1, IC6 MCP23A256, J2 A00-108-220-450, J4 USB-B-S, Q1 12 MHZ

Commit message: Added boxed version and stepped to rev c
Parts:
- added C7: 10uF, rcl:C0805
- added C8, C9: 4.7uF, rcl:C0805
- added IC7: MCP1603, eurosource_mcp1603:SOT23-5L
- added L1: 4.7uH, rcl:L2012C
- added R6, R7: 22, rcl:R0805
- added U$1: (no value), seed_Logo:OSHW_6X150_NOTEXT
- added U$2: (no value), seed_Logo:ROHS_SILK
- added U$3: (no value), VSCP_logo:VSCP_LOGO2
- IC1: value PIC18LF2550-I/SO -> PIC18LF26J50-I/SO
- IC6: value MCP23A256 -> MCP23K256
- moved R1 0.10 mm to (42.7, 29.7)
Connections:
- new net N$13: J4.D-, R6.1
- new net N$14: J4.D+, R7.1
- new net N$16: IC7.5, L1.1
- new net VDD: C2.2, C5.2, C7.2, C9.2, IC1.20, IC1.6, IC6.7, IC6.8, IC7.4, JP4.2, L1.2, R2.2
- net GND: now also C7.1, C8.1, C9.1, IC7.2
- net N$1: now also R7.2; no longer J4.D+
- net N$3: now also R6.2; no longer J4.D-
- net VCC: now also C8.2, IC7.1, IC7.3; no longer C2.2, C5.2, IC1.20, IC6.7, IC6.8, JP4.2, R2.2
Routing:
- net VDD: track 0.00 -> 163.5 mm, vias 0 -> 7
- net GND: track 44.6 -> 205.1 mm, vias 11 -> 19
- net VCC: track 206.4 -> 247.5 mm
- net N$13: track 0.00 -> 15.1 mm
- net N$3: track 27.2 -> 14.5 mm, vias 2 -> 0
- net N$9: track 60.3 -> 51.5 mm
- net SYSTEMCLOCK: track 38.4 -> 31.4 mm, vias 0 -> 2
- net N$1: track 25.1 -> 18.7 mm
- net N$14: track 0.00 -> 4.65 mm
- net MCLR: track 37.0 -> 41.4 mm, vias 2 -> 4
- net N$16: track 0.00 -> 3.47 mm
- net CAN_SDI: track 47.7 -> 50.9 mm
- net N$10: track 19.8 -> 21.8 mm, vias 0 -> 2
- net CAN_CS: track 38.9 -> 39.7 mm
Other:
- board size 72 x 42.6 mm -> 75.7 x 42.5 mm
- board text added: "www.grodansparadis.com"
- board text removed: "www.vscp.org"
