File: eagle/can4vscp_usb_rev_B.sch (EAGLE design)
At the start: 29 parts, among them IC1 PIC18LF2550-I/SO, IC2 MCP2515, IC3 MCP2551SN, IC4 ISO1050, IC5 DCDC_MER1, IC6 MCP23A256, J2 A00-108-220-450, J4 USB-B-S, Q1 12 MHZ

Commit message: Added boxed version and stepped to rev c
Parts:
- added C7: 10uF, rcl:C-EUC0805
- added C8, C9: 4.7uF, rcl:C-EUC0805
- added IC7: MCP1603, eurosource_mcp1603:MCP1603
- added L1: 4.7uH, rcl:L-USL2012C
- added R6, R7: 22, rcl:R-EU_R0805
- IC1: value PIC18LF2550-I/SO -> PIC18LF26J50-I/SO
- IC6: value MCP23A256 -> MCP23K256
Connections:
- new net N$13: J4.D-, R6.1
- new net N$14: J4.D+, R7.1
- new net N$16: IC7.LX, L1.1
- new net VDD: C2.2, C5.2, C7.2, C9.2, IC1.RCV/T0CKI/C1OUT/RA4, IC1.VDD, IC6.HOLD, IC6.VCC, IC7.VOUT, JP4.2, L1.2, R2.2
- net GND: now also C7.1, C8.1, C9.1, IC7.GND
- net N$1: now also R7.2; no longer J4.D+
- net N$3: now also R6.2; no longer J4.D-
- net VCC: now also C8.2, IC7./SHDN, IC7.VIN; no longer C2.2, C5.2, IC1.VDD, IC6.HOLD, IC6.VCC, JP4.2, R2.2
Other:
- note added: "VCC - 5V"
- note added: "VDD - 3.3V"
