File: eagle/can4vscp_usb_rev_c.brd (EAGLE design)
At the start: 72.1 x 42.1 mm, 35 parts, among them IC1 PIC18LF26J50-I/SO, IC2 MCP2515, IC3 MCP2551SN, IC6 MCP23K256, IC7 MCP1603, J2 A00-108-220-450, J4 USB-B-S, Q1 12 MHZ

Commit message: Corrected processor type
Parts:
- IC1: value PIC18LF26J50-I/SO -> PIC18LF25K50-I/SO
Changed lines of the file:
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@@
 <attribute name="NAME" x="39.6813" y="1.9986" size="0.6096" layer="25" rot="R90"/>
 </element>
-<element name="IC1" library="microchip-pic18fxx5x" package="SO-28W" value="PIC18LF26J50-I/SO" x="32.4356" y="31.1742" smashed="yes" rot="R90">
+<element name="IC1" library="microchip-pic18fxx5x" package="SO-28W" value="PIC18LF25K50-I/SO" x="32.4356" y="31.1742" smashed="yes" rot="R90">
 <attribute name="NAME" x="34.5171" y="22.6916" size="0.6096" layer="25" ratio="10" rot="R180"/>
 </element>
